Commit message: adding machine vision exercise

File: ros2_SimRealRobotControl/packages/ur5/ros2srrc_ur5_gazebo/urdf/ur5_robotiq_2f85_with_cams.urdf.xacro (robot description, xacro)
@@ -49,4 +49,9 @@
   <!-- Include XACRO-MACRO file of the UR5: -->
   <xacro:include filename="$(find ros2srrc_robots)/ur5/urdf/ur5_macro.urdf.xacro"/>
+ <xacro:include filename="$(find ros2srrc_ur5_gazebo)/urdf/common_properties.xarco"/>
+  <xacro:include filename="$(find ros2srrc_ur5_gazebo)/urdf/cam_on_hand_params.xacro"/>
+  <xacro:include filename="$(find ros2srrc_ur5_gazebo)/urdf/cam_on_hand.xacro"/>
+  <xacro:include filename="$(find ros2srrc_ur5_gazebo)/urdf/cam_on_base_params.xacro"/>
+  <xacro:include filename="$(find ros2srrc_ur5_gazebo)/urdf/cam_on_base.xacro"/>
   <xacro:ur5
     bringup="${bringup}"
@@ -64,5 +69,5 @@
     parent_link="tool0"
   />
-  <!-- Load ROS 2 Control Gazebo Plugin -->
+  <!-- Load ROS 2 Gazebo Plugin -->
   <xacro:unless value="${bringup}">
     <gazebo>
@@ -73,6 +78,4 @@
         <!-- End-Effector Controller (if needed) -->
         <parameters>$(find ros2srrc_endeffectors)/${EE_name}/config/controller.yaml</parameters>
-        <!-- Yamaha Axis Controller -->
-        <parameters>$(find ros2srrc_robots)/ur5/config/just_yamaha_controller.yaml</parameters>
       </plugin>
     </gazebo>
@@ -80,9 +83,9 @@
   <!-- World: LINK -->
   <link name="world"/>
-  <!-- Yamaha axis: LINK -->
-  <link name="yamaha_axis">
+  <!-- Robot Stand: LINK -->
+  <link name='robot_stand'>
     <inertial>
       <origin xyz="0 0 0" rpy="0 0 0"/>
-      <mass value="1"/>
+      <mass value="100"/>
       <inertia ixx="0.01"  ixy="0"  ixz="0" iyy="0.01" iyz="0" izz="0.01" />
     </inertial>
@@ -90,5 +93,5 @@
       <origin xyz="0 0 0" rpy=" 0 0 0"/>
       <geometry>
-        <box size = "2.0 0.3 0.1"/>
+        <box size = "0.2 0.2 1.0"/>
       </geometry>
     </collision>
@@ -96,48 +99,13 @@
       <origin xyz="0 0 0" rpy=" 0 0 0"/>
       <geometry>
-        <box size = "2.0 0.3 0.1"/>
+        <box size = "0.2 0.2 1.0"/>
       </geometry>
     </visual>
   </link>
-  <!-- Robot Small Stand: LINK -->
-  <link name="robot_stand">
-    <inertial>
-      <origin xyz="0 0 0" rpy="0 0 0"/>
-      <mass value="1"/>
-      <inertia ixx="0.01"  ixy="0"  ixz="0" iyy="0.01" iyz="0" izz="0.01" />
-    </inertial>
-    <collision name='collision'>
-      <origin xyz="0 0 0" rpy=" 0 0 0"/>
-      <geometry>
-        <box size = "0.2 0.2 0.06"/>
-      </geometry>
-    </collision>
-    <visual name='chassis_visual'>
-      <origin xyz="0 0 0" rpy=" 0 0 0"/>
-      <geometry>
-        <box size = "0.2 0.2 0.06"/>
-      </geometry>
-      <material name="LightGrey">
-          <color rgba="0.7 0.7 0.7 1.0"/>
-      </material>
-    </visual>
-  </link>
-  <gazebo reference="robot_stand">
-      <mu1>0.1</mu1>
-      <mu2>0.1</mu2>
-  </gazebo>
-  <!-- World fixed Axis: FIXED JOINT -->
+  <!-- Robot Stand: FIXED JOINT -->
   <joint name="world_joint" type="fixed">
     <parent link= "world" />
-    <child link = "yamaha_axis" />
-    <origin xyz="0.0 0.0 0.95" rpy="0.0 0.0 -1.570796" />
-  </joint>
-  <!-- Yamaha Axis: PRISMATIC JOINT -->
-  <joint name="yamaha_joint" type="prismatic">
-    <parent link= "yamaha_axis" />
     <child link = "robot_stand" />
-    <axis xyz="1 0 0"/>
-    <limit lower="-0.9" upper="0.9" velocity="0.05" effort="10"/>
-    <origin xyz="0.0 0.0 0.08" rpy="0.0 0.0 0.0" />
+    <origin xyz="0.0 0.0 0.5" rpy="0.0 0.0 0.0" />
   </joint>
   <!-- Robot Stand: Robot+Stand JOINT -->
@@ -145,15 +113,17 @@
     <parent link= "robot_stand" />
     <child link = "base_link" />
-    <origin xyz="0.0 0.0 0.0305" rpy="0.0 0.0 0.0" />
+    <origin xyz="0.0 0.0 0.501" rpy="0.0 0.0 0.0" />
   </joint>
-  <!-- Yamaha Axis: TRANSMISSION TYPE
-  <transmission name="yamaha_axis_trans">
-      <type>transmission_interface/SimpleTransmission</type>
-      <joint name="yamaha_joint">
-        <hardwareInterface>hardware_interface/PositionJointInterface</hardwareInterface>
-      </joint>
-      <actuator name="yamaha_axis_motor">
-        <mechanicalReduction>1</mechanicalReduction>
-      </actuator>
-  </transmission> -->
+  <!-- ros2srrc_HMI CAMERA -->
+  <xacro:if value="${hmi}">
+    <xacro:include filename="$(find ros2srrc_hmi)/urdf/hmicamera.urdf.xacro"/>
+    <xacro:HMI_camera
+      x="2.5"
+      y="1.50"
+      z="2.0"
+      roll="0.0"
+      pitch="0.35"
+      yaw="-2.6"
+    />
+  </xacro:if>
 </robot>
