Commit message: update self collision bug

File: ros2_SimRealRobotControl/packages/ur5/ros2srrc_ur5_gazebo/urdf/cam_on_hand_params.xacro (robot description, xacro)
@@ -2,5 +2,5 @@
 <robot xmlns:xacro="http://ros.org/wiki/xacro">
     <xacro:property name="cam_hand_px" value="0.0" />
-    <xacro:property name="cam_hand_py" value="-0.07" />
+    <xacro:property name="cam_hand_py" value="-0.1" />
     <xacro:property name="cam_hand_pz" value="-0.05" />
     <xacro:property name="cam_hand_or" value="0" />

File: ros2_SimRealRobotControl/packages/ur5/ros2srrc_ur5_gazebo/urdf/ur5_robotiq_2f85_with_cams.urdf.xacro (robot description, xacro)
@@ -113,5 +113,5 @@
     <parent link= "robot_stand" />
     <child link = "base_link" />
-    <origin xyz="0.0 0.0 0.501" rpy="0.0 0.0 0.0" />
+    <origin xyz="0.0 0.0 0.52" rpy="0.0 0.0 0.0" />
   </joint>
   <!-- ros2srrc_HMI CAMERA -->
