Commit message: update manipulation

File: ros2_SimRealRobotControl/packages/ur5/ros2srrc_ur5_gazebo/urdf/cam_on_base_params.xacro (robot description, xacro)
@@ -3,8 +3,8 @@
     <xacro:property name="cam_base_px" value="1.0" />
     <xacro:property name="cam_base_py" value="0.0" />
-    <xacro:property name="cam_base_pz" value="0.4" />
+    <xacro:property name="cam_base_pz" value="1.4" />
     <xacro:property name="cam_base_or" value="0.0" />
     <xacro:property name="cam_base_op" value="${pi/4}" />
     <xacro:property name="cam_base_oy" value="${pi}" />
-    <xacro:property name="parent_base" value="base_link" />
+    <xacro:property name="parent_base" value="world" />
 </robot>

File: ros2_SimRealRobotControl/packages/ur5/ros2srrc_ur5_gazebo/urdf/cam_on_hand_params.xacro (robot description, xacro)
@@ -2,6 +2,6 @@
 <robot xmlns:xacro="http://ros.org/wiki/xacro">
     <xacro:property name="cam_hand_px" value="0.0" />
-    <xacro:property name="cam_hand_py" value="-0.1" />
-    <xacro:property name="cam_hand_pz" value="-0.05" />
+    <xacro:property name="cam_hand_py" value="-0.067" />
+    <xacro:property name="cam_hand_pz" value="0.03" />
     <xacro:property name="cam_hand_or" value="0" />
     <xacro:property name="cam_hand_op" value="-1.57" />

File: ros2_SimRealRobotControl/packages/ur5/ros2srrc_ur5_gazebo/urdf/ur5_robotiq_2f85_with_cams.urdf.xacro (robot description, xacro)
@@ -49,5 +49,5 @@
   <!-- Include XACRO-MACRO file of the UR5: -->
   <xacro:include filename="$(find ros2srrc_robots)/ur5/urdf/ur5_macro.urdf.xacro"/>
- <xacro:include filename="$(find ros2srrc_ur5_gazebo)/urdf/common_properties.xarco"/>
+  <xacro:include filename="$(find ros2srrc_ur5_gazebo)/urdf/common_properties.xarco"/>
   <xacro:include filename="$(find ros2srrc_ur5_gazebo)/urdf/cam_on_hand_params.xacro"/>
   <xacro:include filename="$(find ros2srrc_ur5_gazebo)/urdf/cam_on_hand.xacro"/>
