Commit message: update color and shape filter

File: ros2_SimRealRobotControl/packages/ur5/ros2srrc_ur5_gazebo/urdf/cam_on_base.xacro (robot description, xacro)
@@ -50,7 +50,7 @@
             <update_rate>10</update_rate>
             <camera>
-                <horizontal_fov>1.089</horizontal_fov>
+                <horizontal_fov>1.047</horizontal_fov>
                 <image>
-                    <format>R8G8B8</format>
+                    <format>B8G8R8</format>
                     <width>640</width>
                     <height>480</height>

File: ros2_SimRealRobotControl/packages/ur5/ros2srrc_ur5_gazebo/urdf/cam_on_hand.xacro (robot description, xacro)
@@ -49,7 +49,7 @@
             <update_rate>10</update_rate>
             <camera>
-                <horizontal_fov>1.089</horizontal_fov>
+                <horizontal_fov>1.047</horizontal_fov>
                 <image>
-                    <format>R8G8B8</format>
+                    <format>B8G8R8</format>
                     <width>640</width>
                     <height>480</height>

File: ros2_SimRealRobotControl/packages/ur5/ros2srrc_ur5_gazebo/urdf/ur5.urdf.xacro (robot description, xacro)
@@ -88,4 +88,7 @@
         <box size = "0.2 0.2 1.0"/>
       </geometry>
+      <material name="stand_grey">
+        <color rgba="0.2 0.2 0.2 1.0"/>
+      </material>
     </visual>
   </link>

Commit message: fix path issue for docker

File: ros2_SimRealRobotControl/packages/ur5/ros2srrc_ur5_gazebo/urdf/cam_on_base.xacro (robot description, xacro)
@@ -12,5 +12,5 @@
             <geometry>
                 <!-- <box size="0.01 0.03 0.03" /> -->
-                <mesh filename="package://ros2srrc_ur5_gazebo/meshes/kinetic.stl"/>
+                <mesh filename="file://$(find ros2srrc_ur5_gazebo)/meshes/kinetic.stl"/>
             </geometry>
             <material name="dark_grey"/>
@@ -18,5 +18,5 @@
         <collision>
             <geometry>
-                <mesh filename="package://ros2srrc_ur5_gazebo/meshes/kinetic.dae"/>
+                <mesh filename="file://$(find ros2srrc_ur5_gazebo)/meshes/kinetic.dae"/>
             </geometry>
         </collision>
@@ -39,5 +39,5 @@
             <geometry>
                 <mesh>
-                    <uri>package://ros2srrc_ur5_gazebo/meshes/kinetic.stl</uri>
+                    <mesh filename="file://$(find ros2srrc_ur5_gazebo)/meshes/kinetic.stl"/>
                 </mesh>
             </geometry>
@@ -69,5 +69,5 @@
         <visual>
             <geometry>
-                <mesh filename="package://ros2srrc_ur5_gazebo/meshes/kinetic.stl"/>
+                <mesh filename="file://$(find ros2srrc_ur5_gazebo)/meshes/kinetic.stl"/>
             </geometry>
             <material>Gazebo/Red</material>

File: ros2_SimRealRobotControl/packages/ur5/ros2srrc_ur5_gazebo/urdf/cam_on_hand.xacro (robot description, xacro)
@@ -12,5 +12,5 @@
             <geometry>
                 <!-- <box size="0.01 0.03 0.03" /> -->
-                <mesh filename="package://ros2srrc_ur5_gazebo/meshes/kinetic.stl"/>
+                <mesh filename="file://$(find ros2srrc_ur5_gazebo)/meshes/kinetic.stl"/>
             </geometry>
             <material name="dark_grey"/>
@@ -18,5 +18,5 @@
         <collision>
             <geometry>
-                <mesh filename="package://ros2srrc_ur5_gazebo/meshes/kinetic.dae"/>
+                <mesh filename="file://$(find ros2srrc_ur5_gazebo)/meshes/kinetic.dae"/>
             </geometry>
         </collision>
@@ -39,5 +39,5 @@
             <geometry>
                 <mesh>
-                    <uri>package://ros2srrc_ur5_gazebo/meshes/kinetic.stl</uri>
+                    <mesh filename="file://$(find ros2srrc_ur5_gazebo)/meshes/kinetic.stl"/>
                 </mesh>
             </geometry>
@@ -68,5 +68,5 @@
         <visual>
             <geometry>
-                <mesh filename="package://ros2srrc_ur5_gazebo/meshes/kinetic.stl"/>
+                <mesh filename="file://$(find ros2srrc_ur5_gazebo)/meshes/kinetic.stl"/>
             </geometry>
             <material>Gazebo/Red</material>

File: ros2_SimRealRobotControl/packages/ur5/ros2srrc_ur5_gazebo/urdf/ur5_robotiq_2f85_with_cams.urdf.xacro (robot description, xacro)
@@ -49,5 +49,5 @@
   <!-- Include XACRO-MACRO file of the UR5: -->
   <xacro:include filename="$(find ros2srrc_robots)/ur5/urdf/ur5_macro.urdf.xacro"/>
-  <xacro:include filename="$(find ros2srrc_ur5_gazebo)/urdf/common_properties.xarco"/>
+  <xacro:include filename="$(find ros2srrc_ur5_gazebo)/urdf/common_properties.xacro"/>
   <xacro:include filename="$(find ros2srrc_ur5_gazebo)/urdf/cam_on_hand_params.xacro"/>
   <xacro:include filename="$(find ros2srrc_ur5_gazebo)/urdf/cam_on_hand.xacro"/>
